Commit message: Update rope for x-y-rotation and create spinning reward

File: rope.urdf (robot description, URDF)
Before this commit: robot panda, 57 links, 56 joints
Links:
- removed link panda_hand
- removed link panda_link0
- removed link panda_link1
- removed link panda_link2
- removed link panda_link3
- removed link panda_link4
- removed link panda_link5
- removed link panda_link6
- removed link panda_link7
Joints:
- removed joint panda_hand_joint
- removed joint panda_joint1
- removed joint panda_joint2
- removed joint panda_joint3
- removed joint panda_joint4
- removed joint panda_joint5
- removed joint panda_joint6
- removed joint panda_joint7

Commit message: Working rope-end-static

File: rope.urdf (robot description, URDF)
Before this commit: robot rope, 48 links, 48 joints
Links:
- link link1: geometry collision cylinder length=0.041666666666666664 radius=0.02; visual cylinder length=0.041666666666666664 radius=0.02
- link link11: geometry collision cylinder length=0.041666666666666664 radius=0.02; visual cylinder length=0.041666666666666664 radius=0.02
- link link13: geometry collision cylinder length=0.041666666666666664 radius=0.02; visual cylinder length=0.041666666666666664 radius=0.02
- link link15: geometry collision cylinder length=0.041666666666666664 radius=0.02; visual cylinder length=0.041666666666666664 radius=0.02
- link link17: geometry collision cylinder length=0.041666666666666664 radius=0.02; visual cylinder length=0.041666666666666664 radius=0.02
- link link19: geometry collision cylinder length=0.041666666666666664 radius=0.02; visual cylinder length=0.041666666666666664 radius=0.02
- link link21: geometry collision cylinder length=0.041666666666666664 radius=0.02; visual cylinder length=0.041666666666666664 radius=0.02
- link link23: geometry collision cylinder length=0.041666666666666664 radius=0.02; visual cylinder length=0.041666666666666664 radius=0.02
- link link25: geometry collision cylinder length=0.041666666666666664 radius=0.02; visual cylinder length=0.041666666666666664 radius=0.02
- link link27: geometry collision cylinder length=0.041666666666666664 radius=0.02; visual cylinder length=0.041666666666666664 radius=0.02
- link link29: geometry collision cylinder length=0.041666666666666664 radius=0.02; visual cylinder length=0.041666666666666664 radius=0.02
- link link3: geometry collision cylinder length=0.041666666666666664 radius=0.02; visual cylinder length=0.041666666666666664 radius=0.02
- link link31: geometry collision cylinder length=0.041666666666666664 radius=0.02; visual cylinder length=0.041666666666666664 radius=0.02
- link link33: geometry collision cylinder length=0.041666666666666664 radius=0.02; visual cylinder length=0.041666666666666664 radius=0.02
- link link35: geometry collision cylinder length=0.041666666666666664 radius=0.02; visual cylinder length=0.041666666666666664 radius=0.02
- link link37: geometry collision cylinder length=0.041666666666666664 radius=0.02; visual cylinder length=0.041666666666666664 radius=0.02
- link link39: geometry collision cylinder length=0.041666666666666664 radius=0.02; visual cylinder length=0.041666666666666664 radius=0.02
- link link41: geometry collision cylinder length=0.041666666666666664 radius=0.02; visual cylinder length=0.041666666666666664 radius=0.02
- link link43: geometry collision cylinder length=0.041666666666666664 radius=0.02; visual cylinder length=0.041666666666666664 radius=0.02
- link link45: geometry collision cylinder length=0.041666666666666664 radius=0.02; visual cylinder length=0.041666666666666664 radius=0.02
- link link47: geometry collision cylinder length=0.041666666666666664 radius=0.02; visual cylinder length=0.041666666666666664 radius=0.02
- link link5: geometry collision cylinder length=0.041666666666666664 radius=0.02; visual cylinder length=0.041666666666666664 radius=0.02
- link link7: geometry collision cylinder length=0.041666666666666664 radius=0.02; visual cylinder length=0.041666666666666664 radius=0.02
- link link9: geometry collision cylinder length=0.041666666666666664 radius=0.02; visual cylinder length=0.041666666666666664 radius=0.02
Joints:
- joint joint10: origin xyz=0.0 0.0 0.020833333333333332 -> xyz=0.0 0.0 0.041666666666666664
- joint joint12: origin xyz=0.0 0.0 0.020833333333333332 -> xyz=0.0 0.0 0.041666666666666664
- joint joint14: origin xyz=0.0 0.0 0.020833333333333332 -> xyz=0.0 0.0 0.041666666666666664
- joint joint16: origin xyz=0.0 0.0 0.020833333333333332 -> xyz=0.0 0.0 0.041666666666666664
- joint joint18: origin xyz=0.0 0.0 0.020833333333333332 -> xyz=0.0 0.0 0.041666666666666664
- joint joint2: origin xyz=0.0 0.0 0.020833333333333332 -> xyz=0.0 0.0 0.041666666666666664
- joint joint20: origin xyz=0.0 0.0 0.020833333333333332 -> xyz=0.0 0.0 0.041666666666666664
- joint joint22: origin xyz=0.0 0.0 0.020833333333333332 -> xyz=0.0 0.0 0.041666666666666664
- joint joint24: origin xyz=0.0 0.0 0.020833333333333332 -> xyz=0.0 0.0 0.041666666666666664
- joint joint26: origin xyz=0.0 0.0 0.020833333333333332 -> xyz=0.0 0.0 0.041666666666666664
- joint joint28: origin xyz=0.0 0.0 0.020833333333333332 -> xyz=0.0 0.0 0.041666666666666664
- joint joint30: origin xyz=0.0 0.0 0.020833333333333332 -> xyz=0.0 0.0 0.041666666666666664
- joint joint32: origin xyz=0.0 0.0 0.020833333333333332 -> xyz=0.0 0.0 0.041666666666666664
- joint joint34: origin xyz=0.0 0.0 0.020833333333333332 -> xyz=0.0 0.0 0.041666666666666664
- joint joint36: origin xyz=0.0 0.0 0.020833333333333332 -> xyz=0.0 0.0 0.041666666666666664
- joint joint38: origin xyz=0.0 0.0 0.020833333333333332 -> xyz=0.0 0.0 0.041666666666666664
- joint joint4: origin xyz=0.0 0.0 0.020833333333333332 -> xyz=0.0 0.0 0.041666666666666664
- joint joint40: origin xyz=0.0 0.0 0.020833333333333332 -> xyz=0.0 0.0 0.041666666666666664
- joint joint42: origin xyz=0.0 0.0 0.020833333333333332 -> xyz=0.0 0.0 0.041666666666666664
- joint joint44: origin xyz=0.0 0.0 0.020833333333333332 -> xyz=0.0 0.0 0.041666666666666664
- joint joint46: origin xyz=0.0 0.0 0.020833333333333332 -> xyz=0.0 0.0 0.041666666666666664
- joint joint6: origin xyz=0.0 0.0 0.020833333333333332 -> xyz=0.0 0.0 0.041666666666666664
- joint joint8: origin xyz=0.0 0.0 0.020833333333333332 -> xyz=0.0 0.0 0.041666666666666664
