Commit message: Change Rope to have Spherical Joint

File: rope.urdf (robot description, URDF)
Before this commit: robot rope, 48 links, 48 joints
Links:
- link link0: mass 0.0062499999999999995 -> 0.012499999999999999; geometry collision cylinder length=0 radius=0.02; visual cylinder length=0 radius=0.02
- link link1: mass 0.0062499999999999995 -> 0.012499999999999999; geometry collision cylinder length=0.041666666666666664 radius=0.02; visual cylinder length=0.041666666666666664 radius=0.02
- link link10: mass 0.0062499999999999995 -> 0.012499999999999999; geometry collision cylinder length=0 radius=0.02; visual cylinder length=0 radius=0.02
- link link11: mass 0.0062499999999999995 -> 0.012499999999999999; geometry collision cylinder length=0.041666666666666664 radius=0.02; visual cylinder length=0.041666666666666664 radius=0.02
- link link12: mass 0.0062499999999999995 -> 0.012499999999999999; geometry collision cylinder length=0 radius=0.02; visual cylinder length=0 radius=0.02
- link link13: mass 0.0062499999999999995 -> 0.012499999999999999; geometry collision cylinder length=0.041666666666666664 radius=0.02; visual cylinder length=0.041666666666666664 radius=0.02
- link link14: mass 0.0062499999999999995 -> 0.012499999999999999; geometry collision cylinder length=0 radius=0.02; visual cylinder length=0 radius=0.02
- link link15: mass 0.0062499999999999995 -> 0.012499999999999999; geometry collision cylinder length=0.041666666666666664 radius=0.02; visual cylinder length=0.041666666666666664 radius=0.02
- link link16: mass 0.0062499999999999995 -> 0.012499999999999999; geometry collision cylinder length=0 radius=0.02; visual cylinder length=0 radius=0.02
- link link17: mass 0.0062499999999999995 -> 0.012499999999999999; geometry collision cylinder length=0.041666666666666664 radius=0.02; visual cylinder length=0.041666666666666664 radius=0.02
- link link18: mass 0.0062499999999999995 -> 0.012499999999999999; geometry collision cylinder length=0 radius=0.02; visual cylinder length=0 radius=0.02
- link link19: mass 0.0062499999999999995 -> 0.012499999999999999; geometry collision cylinder length=0.041666666666666664 radius=0.02; visual cylinder length=0.041666666666666664 radius=0.02
- link link2: mass 0.0062499999999999995 -> 0.012499999999999999; geometry collision cylinder length=0 radius=0.02; visual cylinder length=0 radius=0.02
- link link20: mass 0.0062499999999999995 -> 0.012499999999999999; geometry collision cylinder length=0 radius=0.02; visual cylinder length=0 radius=0.02
- link link21: mass 0.0062499999999999995 -> 0.012499999999999999; geometry collision cylinder length=0.041666666666666664 radius=0.02; visual cylinder length=0.041666666666666664 radius=0.02
- link link22: mass 0.0062499999999999995 -> 0.012499999999999999; geometry collision cylinder length=0 radius=0.02; visual cylinder length=0 radius=0.02
- link link23: mass 0.0062499999999999995 -> 0.012499999999999999; geometry collision cylinder length=0.041666666666666664 radius=0.02; visual cylinder length=0.041666666666666664 radius=0.02
- link link24: mass 0.0062499999999999995 -> 0.012499999999999999; geometry collision cylinder length=0 radius=0.02; visual cylinder length=0 radius=0.02
- link link25: mass 0.0062499999999999995 -> 0.012499999999999999; geometry collision cylinder length=0.041666666666666664 radius=0.02; visual cylinder length=0.041666666666666664 radius=0.02
- link link26: mass 0.0062499999999999995 -> 0.012499999999999999; geometry collision cylinder length=0 radius=0.02; visual cylinder length=0 radius=0.02
- link link27: mass 0.0062499999999999995 -> 0.012499999999999999; geometry collision cylinder length=0.041666666666666664 radius=0.02; visual cylinder length=0.041666666666666664 radius=0.02
- link link28: mass 0.0062499999999999995 -> 0.012499999999999999; geometry collision cylinder length=0 radius=0.02; visual cylinder length=0 radius=0.02
- link link29: mass 0.0062499999999999995 -> 0.012499999999999999; geometry collision cylinder length=0.041666666666666664 radius=0.02; visual cylinder length=0.041666666666666664 radius=0.02
- link link3: mass 0.0062499999999999995 -> 0.012499999999999999; geometry collision cylinder length=0.041666666666666664 radius=0.02; visual cylinder length=0.041666666666666664 radius=0.02
- link link30: mass 0.0062499999999999995 -> 0.012499999999999999; geometry collision cylinder length=0 radius=0.02; visual cylinder length=0 radius=0.02
- link link31: mass 0.0062499999999999995 -> 0.012499999999999999; geometry collision cylinder length=0.041666666666666664 radius=0.02; visual cylinder length=0.041666666666666664 radius=0.02
- link link32: mass 0.0062499999999999995 -> 0.012499999999999999; geometry collision cylinder length=0 radius=0.02; visual cylinder length=0 radius=0.02
- link link33: mass 0.0062499999999999995 -> 0.012499999999999999; geometry collision cylinder length=0.041666666666666664 radius=0.02; visual cylinder length=0.041666666666666664 radius=0.02
- link link34: mass 0.0062499999999999995 -> 0.012499999999999999; geometry collision cylinder length=0 radius=0.02; visual cylinder length=0 radius=0.02
- link link35: mass 0.0062499999999999995 -> 0.012499999999999999; geometry collision cylinder length=0.041666666666666664 radius=0.02; visual cylinder length=0.041666666666666664 radius=0.02
- link link36: mass 0.0062499999999999995 -> 0.012499999999999999; geometry collision cylinder length=0 radius=0.02; visual cylinder length=0 radius=0.02
- link link37: mass 0.0062499999999999995 -> 0.012499999999999999; geometry collision cylinder length=0.041666666666666664 radius=0.02; visual cylinder length=0.041666666666666664 radius=0.02
- link link38: mass 0.0062499999999999995 -> 0.012499999999999999; geometry collision cylinder length=0 radius=0.02; visual cylinder length=0 radius=0.02
- link link39: mass 0.0062499999999999995 -> 0.012499999999999999; geometry collision cylinder length=0.041666666666666664 radius=0.02; visual cylinder length=0.041666666666666664 radius=0.02
- link link4: mass 0.0062499999999999995 -> 0.012499999999999999; geometry collision cylinder length=0 radius=0.02; visual cylinder length=0 radius=0.02
- link link40: mass 0.0062499999999999995 -> 0.012499999999999999; geometry collision cylinder length=0 radius=0.02; visual cylinder length=0 radius=0.02
- link link41: mass 0.0062499999999999995 -> 0.012499999999999999; geometry collision cylinder length=0.041666666666666664 radius=0.02; visual cylinder length=0.041666666666666664 radius=0.02
- link link42: mass 0.0062499999999999995 -> 0.012499999999999999; geometry collision cylinder length=0 radius=0.02; visual cylinder length=0 radius=0.02
- link link43: mass 0.0062499999999999995 -> 0.012499999999999999; geometry collision cylinder length=0.041666666666666664 radius=0.02; visual cylinder length=0.041666666666666664 radius=0.02
- link link44: mass 0.0062499999999999995 -> 0.012499999999999999; geometry collision cylinder length=0 radius=0.02; visual cylinder length=0 radius=0.02
- link link45: mass 0.0062499999999999995 -> 0.012499999999999999; geometry collision cylinder length=0.041666666666666664 radius=0.02; visual cylinder length=0.041666666666666664 radius=0.02
- link link46: mass 0.0062499999999999995 -> 0.012499999999999999; geometry collision cylinder length=0 radius=0.02; visual cylinder length=0 radius=0.02
- link link47: mass 0.0062499999999999995 -> 0.012499999999999999; geometry collision cylinder length=0.041666666666666664 radius=0.02; visual cylinder length=0.041666666666666664 radius=0.02
- link link5: mass 0.0062499999999999995 -> 0.012499999999999999; geometry collision cylinder length=0.041666666666666664 radius=0.02; visual cylinder length=0.041666666666666664 radius=0.02
- link link6: mass 0.0062499999999999995 -> 0.012499999999999999; geometry collision cylinder length=0 radius=0.02; visual cylinder length=0 radius=0.02
- link link7: mass 0.0062499999999999995 -> 0.012499999999999999; geometry collision cylinder length=0.041666666666666664 radius=0.02; visual cylinder length=0.041666666666666664 radius=0.02
- link link8: mass 0.0062499999999999995 -> 0.012499999999999999; geometry collision cylinder length=0 radius=0.02; visual cylinder length=0 radius=0.02
- link link9: mass 0.0062499999999999995 -> 0.012499999999999999; geometry collision cylinder length=0.041666666666666664 radius=0.02; visual cylinder length=0.041666666666666664 radius=0.02
Joints:
- joint joint1: origin xyz=0.0 0.0 0.020833333333333332 -> xyz=0.0 0.0 0
- joint joint10: origin xyz=0.0 0.0 0.020833333333333332 -> xyz=0.0 0.0 0.041666666666666664
- joint joint11: origin xyz=0.0 0.0 0.020833333333333332 -> xyz=0.0 0.0 0
- joint joint12: origin xyz=0.0 0.0 0.020833333333333332 -> xyz=0.0 0.0 0.041666666666666664
- joint joint13: origin xyz=0.0 0.0 0.020833333333333332 -> xyz=0.0 0.0 0
- joint joint14: origin xyz=0.0 0.0 0.020833333333333332 -> xyz=0.0 0.0 0.041666666666666664
- joint joint15: origin xyz=0.0 0.0 0.020833333333333332 -> xyz=0.0 0.0 0
- joint joint16: origin xyz=0.0 0.0 0.020833333333333332 -> xyz=0.0 0.0 0.041666666666666664
- joint joint17: origin xyz=0.0 0.0 0.020833333333333332 -> xyz=0.0 0.0 0
- joint joint18: origin xyz=0.0 0.0 0.020833333333333332 -> xyz=0.0 0.0 0.041666666666666664
- joint joint19: origin xyz=0.0 0.0 0.020833333333333332 -> xyz=0.0 0.0 0
- joint joint2: origin xyz=0.0 0.0 0.020833333333333332 -> xyz=0.0 0.0 0.041666666666666664
- joint joint20: origin xyz=0.0 0.0 0.020833333333333332 -> xyz=0.0 0.0 0.041666666666666664
- joint joint21: origin xyz=0.0 0.0 0.020833333333333332 -> xyz=0.0 0.0 0
- joint joint22: origin xyz=0.0 0.0 0.020833333333333332 -> xyz=0.0 0.0 0.041666666666666664
- joint joint23: origin xyz=0.0 0.0 0.020833333333333332 -> xyz=0.0 0.0 0
- joint joint24: origin xyz=0.0 0.0 0.020833333333333332 -> xyz=0.0 0.0 0.041666666666666664
- joint joint25: origin xyz=0.0 0.0 0.020833333333333332 -> xyz=0.0 0.0 0
- joint joint26: origin xyz=0.0 0.0 0.020833333333333332 -> xyz=0.0 0.0 0.041666666666666664
- joint joint27: origin xyz=0.0 0.0 0.020833333333333332 -> xyz=0.0 0.0 0
- joint joint28: origin xyz=0.0 0.0 0.020833333333333332 -> xyz=0.0 0.0 0.041666666666666664
- joint joint29: origin xyz=0.0 0.0 0.020833333333333332 -> xyz=0.0 0.0 0
- joint joint3: origin xyz=0.0 0.0 0.020833333333333332 -> xyz=0.0 0.0 0
- joint joint30: origin xyz=0.0 0.0 0.020833333333333332 -> xyz=0.0 0.0 0.041666666666666664
- joint joint31: origin xyz=0.0 0.0 0.020833333333333332 -> xyz=0.0 0.0 0
- joint joint32: origin xyz=0.0 0.0 0.020833333333333332 -> xyz=0.0 0.0 0.041666666666666664
- joint joint33: origin xyz=0.0 0.0 0.020833333333333332 -> xyz=0.0 0.0 0
- joint joint34: origin xyz=0.0 0.0 0.020833333333333332 -> xyz=0.0 0.0 0.041666666666666664
- joint joint35: origin xyz=0.0 0.0 0.020833333333333332 -> xyz=0.0 0.0 0
- joint joint36: origin xyz=0.0 0.0 0.020833333333333332 -> xyz=0.0 0.0 0.041666666666666664
- joint joint37: origin xyz=0.0 0.0 0.020833333333333332 -> xyz=0.0 0.0 0
- joint joint38: origin xyz=0.0 0.0 0.020833333333333332 -> xyz=0.0 0.0 0.041666666666666664
- joint joint39: origin xyz=0.0 0.0 0.020833333333333332 -> xyz=0.0 0.0 0
- joint joint4: origin xyz=0.0 0.0 0.020833333333333332 -> xyz=0.0 0.0 0.041666666666666664
- joint joint40: origin xyz=0.0 0.0 0.020833333333333332 -> xyz=0.0 0.0 0.041666666666666664
- joint joint41: origin xyz=0.0 0.0 0.020833333333333332 -> xyz=0.0 0.0 0
- joint joint42: origin xyz=0.0 0.0 0.020833333333333332 -> xyz=0.0 0.0 0.041666666666666664
- joint joint43: origin xyz=0.0 0.0 0.020833333333333332 -> xyz=0.0 0.0 0
- joint joint44: origin xyz=0.0 0.0 0.020833333333333332 -> xyz=0.0 0.0 0.041666666666666664
- joint joint45: origin xyz=0.0 0.0 0.020833333333333332 -> xyz=0.0 0.0 0
- joint joint46: origin xyz=0.0 0.0 0.020833333333333332 -> xyz=0.0 0.0 0.041666666666666664
- joint joint47: origin xyz=0.0 0.0 0.020833333333333332 -> xyz=0.0 0.0 0
- joint joint5: origin xyz=0.0 0.0 0.020833333333333332 -> xyz=0.0 0.0 0
- joint joint6: origin xyz=0.0 0.0 0.020833333333333332 -> xyz=0.0 0.0 0.041666666666666664
- joint joint7: origin xyz=0.0 0.0 0.020833333333333332 -> xyz=0.0 0.0 0
- joint joint8: origin xyz=0.0 0.0 0.020833333333333332 -> xyz=0.0 0.0 0.041666666666666664
- joint joint9: origin xyz=0.0 0.0 0.020833333333333332 -> xyz=0.0 0.0 0

Commit message: Modify UR5RopePPO's default minibatch setting for smooth laptop debugging

File: assets/urdf/franka_description/robots/franka_panda_rope.urdf (robot description, URDF)
Before this commit: robot panda, 57 links, 56 joints
Links:
- link link0: geometry collision cylinder length=0 radius=0; visual cylinder length=0 radius=0
- link link10: geometry collision cylinder length=0 radius=0; visual cylinder length=0 radius=0
- link link12: geometry collision cylinder length=0 radius=0; visual cylinder length=0 radius=0
- link link14: geometry collision cylinder length=0 radius=0; visual cylinder length=0 radius=0
- link link16: geometry collision cylinder length=0 radius=0; visual cylinder length=0 radius=0
- link link18: geometry collision cylinder length=0 radius=0; visual cylinder length=0 radius=0
- link link2: geometry collision cylinder length=0 radius=0; visual cylinder length=0 radius=0
- link link20: geometry collision cylinder length=0 radius=0; visual cylinder length=0 radius=0
- link link22: geometry collision cylinder length=0 radius=0; visual cylinder length=0 radius=0
- link link24: geometry collision cylinder length=0 radius=0; visual cylinder length=0 radius=0
- link link26: geometry collision cylinder length=0 radius=0; visual cylinder length=0 radius=0
- link link28: geometry collision cylinder length=0 radius=0; visual cylinder length=0 radius=0
- link link30: geometry collision cylinder length=0 radius=0; visual cylinder length=0 radius=0
- link link32: geometry collision cylinder length=0 radius=0; visual cylinder length=0 radius=0
- link link34: geometry collision cylinder length=0 radius=0; visual cylinder length=0 radius=0
- link link36: geometry collision cylinder length=0 radius=0; visual cylinder length=0 radius=0
- link link38: geometry collision cylinder length=0 radius=0; visual cylinder length=0 radius=0
- link link4: geometry collision cylinder length=0 radius=0; visual cylinder length=0 radius=0
- link link40: geometry collision cylinder length=0 radius=0; visual cylinder length=0 radius=0
- link link42: geometry collision cylinder length=0 radius=0; visual cylinder length=0 radius=0
- link link44: geometry collision cylinder length=0 radius=0; visual cylinder length=0 radius=0
- link link46: geometry collision cylinder length=0 radius=0; visual cylinder length=0 radius=0
- link link6: geometry collision cylinder length=0 radius=0; visual cylinder length=0 radius=0
- link link8: geometry collision cylinder length=0 radius=0; visual cylinder length=0 radius=0

File: rope.urdf (robot description, URDF)
Before this commit: robot rope, 48 links, 48 joints
Links:
- link link0: geometry collision cylinder length=0 radius=0; visual cylinder length=0 radius=0
- link link10: geometry collision cylinder length=0 radius=0; visual cylinder length=0 radius=0
- link link12: geometry collision cylinder length=0 radius=0; visual cylinder length=0 radius=0
- link link14: geometry collision cylinder length=0 radius=0; visual cylinder length=0 radius=0
- link link16: geometry collision cylinder length=0 radius=0; visual cylinder length=0 radius=0
- link link18: geometry collision cylinder length=0 radius=0; visual cylinder length=0 radius=0
- link link2: geometry collision cylinder length=0 radius=0; visual cylinder length=0 radius=0
- link link20: geometry collision cylinder length=0 radius=0; visual cylinder length=0 radius=0
- link link22: geometry collision cylinder length=0 radius=0; visual cylinder length=0 radius=0
- link link24: geometry collision cylinder length=0 radius=0; visual cylinder length=0 radius=0
- link link26: geometry collision cylinder length=0 radius=0; visual cylinder length=0 radius=0
- link link28: geometry collision cylinder length=0 radius=0; visual cylinder length=0 radius=0
- link link30: geometry collision cylinder length=0 radius=0; visual cylinder length=0 radius=0
- link link32: geometry collision cylinder length=0 radius=0; visual cylinder length=0 radius=0
- link link34: geometry collision cylinder length=0 radius=0; visual cylinder length=0 radius=0
- link link36: geometry collision cylinder length=0 radius=0; visual cylinder length=0 radius=0
- link link38: geometry collision cylinder length=0 radius=0; visual cylinder length=0 radius=0
- link link4: geometry collision cylinder length=0 radius=0; visual cylinder length=0 radius=0
- link link40: geometry collision cylinder length=0 radius=0; visual cylinder length=0 radius=0
- link link42: geometry collision cylinder length=0 radius=0; visual cylinder length=0 radius=0
- link link44: geometry collision cylinder length=0 radius=0; visual cylinder length=0 radius=0
- link link46: geometry collision cylinder length=0 radius=0; visual cylinder length=0 radius=0
- link link6: geometry collision cylinder length=0 radius=0; visual cylinder length=0 radius=0
- link link8: geometry collision cylinder length=0 radius=0; visual cylinder length=0 radius=0
