Commit message: Fix Rope urdf by removing jointlimit

File: assets/urdf/franka_description/robots/franka_panda_rope.urdf (robot description, URDF)
Before this commit: robot panda, 57 links, 56 joints
Joints:
- joint joint0: limit lower=-2.5 upper=2.5 effort=20 velocity=20 -> (none)
- joint joint1: limit lower=-2.5 upper=2.5 effort=20 velocity=20 -> (none)
- joint joint10: limit lower=-2.5 upper=2.5 effort=20 velocity=20 -> (none)
- joint joint11: limit lower=-2.5 upper=2.5 effort=20 velocity=20 -> (none)
- joint joint12: limit lower=-2.5 upper=2.5 effort=20 velocity=20 -> (none)
- joint joint13: limit lower=-2.5 upper=2.5 effort=20 velocity=20 -> (none)
- joint joint14: limit lower=-2.5 upper=2.5 effort=20 velocity=20 -> (none)
- joint joint15: limit lower=-2.5 upper=2.5 effort=20 velocity=20 -> (none)
- joint joint16: limit lower=-2.5 upper=2.5 effort=20 velocity=20 -> (none)
- joint joint17: limit lower=-2.5 upper=2.5 effort=20 velocity=20 -> (none)
- joint joint18: limit lower=-2.5 upper=2.5 effort=20 velocity=20 -> (none)
- joint joint19: limit lower=-2.5 upper=2.5 effort=20 velocity=20 -> (none)
- joint joint2: limit lower=-2.5 upper=2.5 effort=20 velocity=20 -> (none)
- joint joint20: limit lower=-2.5 upper=2.5 effort=20 velocity=20 -> (none)
- joint joint21: limit lower=-2.5 upper=2.5 effort=20 velocity=20 -> (none)
- joint joint22: limit lower=-2.5 upper=2.5 effort=20 velocity=20 -> (none)
- joint joint23: limit lower=-2.5 upper=2.5 effort=20 velocity=20 -> (none)
- joint joint24: limit lower=-2.5 upper=2.5 effort=20 velocity=20 -> (none)
- joint joint25: limit lower=-2.5 upper=2.5 effort=20 velocity=20 -> (none)
- joint joint26: limit lower=-2.5 upper=2.5 effort=20 velocity=20 -> (none)
- joint joint27: limit lower=-2.5 upper=2.5 effort=20 velocity=20 -> (none)
- joint joint28: limit lower=-2.5 upper=2.5 effort=20 velocity=20 -> (none)
- joint joint29: limit lower=-2.5 upper=2.5 effort=20 velocity=20 -> (none)
- joint joint3: limit lower=-2.5 upper=2.5 effort=20 velocity=20 -> (none)
- joint joint30: limit lower=-2.5 upper=2.5 effort=20 velocity=20 -> (none)
- joint joint31: limit lower=-2.5 upper=2.5 effort=20 velocity=20 -> (none)
- joint joint32: limit lower=-2.5 upper=2.5 effort=20 velocity=20 -> (none)
- joint joint33: limit lower=-2.5 upper=2.5 effort=20 velocity=20 -> (none)
- joint joint34: limit lower=-2.5 upper=2.5 effort=20 velocity=20 -> (none)
- joint joint35: limit lower=-2.5 upper=2.5 effort=20 velocity=20 -> (none)
- joint joint36: limit lower=-2.5 upper=2.5 effort=20 velocity=20 -> (none)
- joint joint37: limit lower=-2.5 upper=2.5 effort=20 velocity=20 -> (none)
- joint joint38: limit lower=-2.5 upper=2.5 effort=20 velocity=20 -> (none)
- joint joint39: limit lower=-2.5 upper=2.5 effort=20 velocity=20 -> (none)
- joint joint4: limit lower=-2.5 upper=2.5 effort=20 velocity=20 -> (none)
- joint joint40: limit lower=-2.5 upper=2.5 effort=20 velocity=20 -> (none)
- joint joint41: limit lower=-2.5 upper=2.5 effort=20 velocity=20 -> (none)
- joint joint42: limit lower=-2.5 upper=2.5 effort=20 velocity=20 -> (none)
- joint joint43: limit lower=-2.5 upper=2.5 effort=20 velocity=20 -> (none)
- joint joint44: limit lower=-2.5 upper=2.5 effort=20 velocity=20 -> (none)
- joint joint45: limit lower=-2.5 upper=2.5 effort=20 velocity=20 -> (none)
- joint joint46: limit lower=-2.5 upper=2.5 effort=20 velocity=20 -> (none)
- joint joint47: limit lower=-2.5 upper=2.5 effort=20 velocity=20 -> (none)
- joint joint5: limit lower=-2.5 upper=2.5 effort=20 velocity=20 -> (none)
- joint joint6: limit lower=-2.5 upper=2.5 effort=20 velocity=20 -> (none)
- joint joint7: limit lower=-2.5 upper=2.5 effort=20 velocity=20 -> (none)
- joint joint8: limit lower=-2.5 upper=2.5 effort=20 velocity=20 -> (none)
- joint joint9: limit lower=-2.5 upper=2.5 effort=20 velocity=20 -> (none)

File: rope.urdf (robot description, URDF)
Before this commit: robot rope, 48 links, 48 joints
Links:
- link link1: geometry collision cylinder length=0.020833333333333332 radius=0.02; visual cylinder length=0.020833333333333332 radius=0.02
- link link11: geometry collision cylinder length=0.020833333333333332 radius=0.02; visual cylinder length=0.020833333333333332 radius=0.02
- link link13: geometry collision cylinder length=0.020833333333333332 radius=0.02; visual cylinder length=0.020833333333333332 radius=0.02
- link link15: geometry collision cylinder length=0.020833333333333332 radius=0.02; visual cylinder length=0.020833333333333332 radius=0.02
- link link17: geometry collision cylinder length=0.020833333333333332 radius=0.02; visual cylinder length=0.020833333333333332 radius=0.02
- link link19: geometry collision cylinder length=0.020833333333333332 radius=0.02; visual cylinder length=0.020833333333333332 radius=0.02
- link link21: geometry collision cylinder length=0.020833333333333332 radius=0.02; visual cylinder length=0.020833333333333332 radius=0.02
- link link23: geometry collision cylinder length=0.020833333333333332 radius=0.02; visual cylinder length=0.020833333333333332 radius=0.02
- link link25: geometry collision cylinder length=0.020833333333333332 radius=0.02; visual cylinder length=0.020833333333333332 radius=0.02
- link link27: geometry collision cylinder length=0.020833333333333332 radius=0.02; visual cylinder length=0.020833333333333332 radius=0.02
- link link29: geometry collision cylinder length=0.020833333333333332 radius=0.02; visual cylinder length=0.020833333333333332 radius=0.02
- link link3: geometry collision cylinder length=0.020833333333333332 radius=0.02; visual cylinder length=0.020833333333333332 radius=0.02
- link link31: geometry collision cylinder length=0.020833333333333332 radius=0.02; visual cylinder length=0.020833333333333332 radius=0.02
- link link33: geometry collision cylinder length=0.020833333333333332 radius=0.02; visual cylinder length=0.020833333333333332 radius=0.02
- link link35: geometry collision cylinder length=0.020833333333333332 radius=0.02; visual cylinder length=0.020833333333333332 radius=0.02
- link link37: geometry collision cylinder length=0.020833333333333332 radius=0.02; visual cylinder length=0.020833333333333332 radius=0.02
- link link39: geometry collision cylinder length=0.020833333333333332 radius=0.02; visual cylinder length=0.020833333333333332 radius=0.02
- link link41: geometry collision cylinder length=0.020833333333333332 radius=0.02; visual cylinder length=0.020833333333333332 radius=0.02
- link link43: geometry collision cylinder length=0.020833333333333332 radius=0.02; visual cylinder length=0.020833333333333332 radius=0.02
- link link45: geometry collision cylinder length=0.020833333333333332 radius=0.02; visual cylinder length=0.020833333333333332 radius=0.02
- link link47: geometry collision cylinder length=0.020833333333333332 radius=0.02; visual cylinder length=0.020833333333333332 radius=0.02
- link link5: geometry collision cylinder length=0.020833333333333332 radius=0.02; visual cylinder length=0.020833333333333332 radius=0.02
- link link7: geometry collision cylinder length=0.020833333333333332 radius=0.02; visual cylinder length=0.020833333333333332 radius=0.02
- link link9: geometry collision cylinder length=0.020833333333333332 radius=0.02; visual cylinder length=0.020833333333333332 radius=0.02
Joints:
- joint joint0: limit lower=-2.5 upper=2.5 effort=20 velocity=20 -> (none)
- joint joint1: limit lower=-2.5 upper=2.5 effort=20 velocity=20 -> (none)
- joint joint10: limit lower=-2.5 upper=2.5 effort=20 velocity=20 -> (none); origin xyz=0.0 0.0 0.041666666666666664 -> xyz=0.0 0.0 0.020833333333333332
- joint joint11: limit lower=-2.5 upper=2.5 effort=20 velocity=20 -> (none)
- joint joint12: limit lower=-2.5 upper=2.5 effort=20 velocity=20 -> (none); origin xyz=0.0 0.0 0.041666666666666664 -> xyz=0.0 0.0 0.020833333333333332
- joint joint13: limit lower=-2.5 upper=2.5 effort=20 velocity=20 -> (none)
- joint joint14: limit lower=-2.5 upper=2.5 effort=20 velocity=20 -> (none); origin xyz=0.0 0.0 0.041666666666666664 -> xyz=0.0 0.0 0.020833333333333332
- joint joint15: limit lower=-2.5 upper=2.5 effort=20 velocity=20 -> (none)
- joint joint16: limit lower=-2.5 upper=2.5 effort=20 velocity=20 -> (none); origin xyz=0.0 0.0 0.041666666666666664 -> xyz=0.0 0.0 0.020833333333333332
- joint joint17: limit lower=-2.5 upper=2.5 effort=20 velocity=20 -> (none)
- joint joint18: limit lower=-2.5 upper=2.5 effort=20 velocity=20 -> (none); origin xyz=0.0 0.0 0.041666666666666664 -> xyz=0.0 0.0 0.020833333333333332
- joint joint19: limit lower=-2.5 upper=2.5 effort=20 velocity=20 -> (none)
- joint joint2: limit lower=-2.5 upper=2.5 effort=20 velocity=20 -> (none); origin xyz=0.0 0.0 0.041666666666666664 -> xyz=0.0 0.0 0.020833333333333332
- joint joint20: limit lower=-2.5 upper=2.5 effort=20 velocity=20 -> (none); origin xyz=0.0 0.0 0.041666666666666664 -> xyz=0.0 0.0 0.020833333333333332
- joint joint21: limit lower=-2.5 upper=2.5 effort=20 velocity=20 -> (none)
- joint joint22: limit lower=-2.5 upper=2.5 effort=20 velocity=20 -> (none); origin xyz=0.0 0.0 0.041666666666666664 -> xyz=0.0 0.0 0.020833333333333332
- joint joint23: limit lower=-2.5 upper=2.5 effort=20 velocity=20 -> (none)
- joint joint24: limit lower=-2.5 upper=2.5 effort=20 velocity=20 -> (none); origin xyz=0.0 0.0 0.041666666666666664 -> xyz=0.0 0.0 0.020833333333333332
- joint joint25: limit lower=-2.5 upper=2.5 effort=20 velocity=20 -> (none)
- joint joint26: limit lower=-2.5 upper=2.5 effort=20 velocity=20 -> (none); origin xyz=0.0 0.0 0.041666666666666664 -> xyz=0.0 0.0 0.020833333333333332
- joint joint27: limit lower=-2.5 upper=2.5 effort=20 velocity=20 -> (none)
- joint joint28: limit lower=-2.5 upper=2.5 effort=20 velocity=20 -> (none); origin xyz=0.0 0.0 0.041666666666666664 -> xyz=0.0 0.0 0.020833333333333332
- joint joint29: limit lower=-2.5 upper=2.5 effort=20 velocity=20 -> (none)
- joint joint3: limit lower=-2.5 upper=2.5 effort=20 velocity=20 -> (none)
- joint joint30: limit lower=-2.5 upper=2.5 effort=20 velocity=20 -> (none); origin xyz=0.0 0.0 0.041666666666666664 -> xyz=0.0 0.0 0.020833333333333332
- joint joint31: limit lower=-2.5 upper=2.5 effort=20 velocity=20 -> (none)
- joint joint32: limit lower=-2.5 upper=2.5 effort=20 velocity=20 -> (none); origin xyz=0.0 0.0 0.041666666666666664 -> xyz=0.0 0.0 0.020833333333333332
- joint joint33: limit lower=-2.5 upper=2.5 effort=20 velocity=20 -> (none)
- joint joint34: limit lower=-2.5 upper=2.5 effort=20 velocity=20 -> (none); origin xyz=0.0 0.0 0.041666666666666664 -> xyz=0.0 0.0 0.020833333333333332
- joint joint35: limit lower=-2.5 upper=2.5 effort=20 velocity=20 -> (none)
- joint joint36: limit lower=-2.5 upper=2.5 effort=20 velocity=20 -> (none); origin xyz=0.0 0.0 0.041666666666666664 -> xyz=0.0 0.0 0.020833333333333332
- joint joint37: limit lower=-2.5 upper=2.5 effort=20 velocity=20 -> (none)
- joint joint38: limit lower=-2.5 upper=2.5 effort=20 velocity=20 -> (none); origin xyz=0.0 0.0 0.041666666666666664 -> xyz=0.0 0.0 0.020833333333333332
- joint joint39: limit lower=-2.5 upper=2.5 effort=20 velocity=20 -> (none)
- joint joint4: limit lower=-2.5 upper=2.5 effort=20 velocity=20 -> (none); origin xyz=0.0 0.0 0.041666666666666664 -> xyz=0.0 0.0 0.020833333333333332
- joint joint40: limit lower=-2.5 upper=2.5 effort=20 velocity=20 -> (none); origin xyz=0.0 0.0 0.041666666666666664 -> xyz=0.0 0.0 0.020833333333333332
- joint joint41: limit lower=-2.5 upper=2.5 effort=20 velocity=20 -> (none)
- joint joint42: limit lower=-2.5 upper=2.5 effort=20 velocity=20 -> (none); origin xyz=0.0 0.0 0.041666666666666664 -> xyz=0.0 0.0 0.020833333333333332
- joint joint43: limit lower=-2.5 upper=2.5 effort=20 velocity=20 -> (none)
- joint joint44: limit lower=-2.5 upper=2.5 effort=20 velocity=20 -> (none); origin xyz=0.0 0.0 0.041666666666666664 -> xyz=0.0 0.0 0.020833333333333332
- joint joint45: limit lower=-2.5 upper=2.5 effort=20 velocity=20 -> (none)
- joint joint46: limit lower=-2.5 upper=2.5 effort=20 velocity=20 -> (none); origin xyz=0.0 0.0 0.041666666666666664 -> xyz=0.0 0.0 0.020833333333333332
- joint joint47: limit lower=-2.5 upper=2.5 effort=20 velocity=20 -> (none)
- joint joint5: limit lower=-2.5 upper=2.5 effort=20 velocity=20 -> (none)
- joint joint6: limit lower=-2.5 upper=2.5 effort=20 velocity=20 -> (none); origin xyz=0.0 0.0 0.041666666666666664 -> xyz=0.0 0.0 0.020833333333333332
- joint joint7: limit lower=-2.5 upper=2.5 effort=20 velocity=20 -> (none)
- joint joint8: limit lower=-2.5 upper=2.5 effort=20 velocity=20 -> (none); origin xyz=0.0 0.0 0.041666666666666664 -> xyz=0.0 0.0 0.020833333333333332
- joint joint9: limit lower=-2.5 upper=2.5 effort=20 velocity=20 -> (none)
