Commit message: Testing Ropes

File: assets/urdf/franka_description/robots/franka_panda_rope.urdf (robot description, URDF)
Before this commit: robot panda, 57 links, 56 joints
Links:
- removed link link24
- removed link link25
- removed link link26
- removed link link27
- removed link link28
- removed link link29
- removed link link30
- removed link link31
- removed link link32
- removed link link33
- removed link link34
- removed link link35
- removed link link36
- removed link link37
- removed link link38
- removed link link39
- removed link link40
- removed link link41
- removed link link42
- removed link link43
- removed link link44
- removed link link45
- removed link link46
- removed link link47
- link link0: mass 0.012499999999999999 -> 0.024999999999999998
- link link1: mass 0.012499999999999999 -> 0.024999999999999998; geometry collision cylinder length=0.04333333333333332 radius=0.01; visual cylinder length=0.04333333333333332 radius=0.01
- link link10: mass 0.012499999999999999 -> 0.024999999999999998
- link link11: mass 0.012499999999999999 -> 0.024999999999999998; geometry collision cylinder length=0.04333333333333332 radius=0.01; visual cylinder length=0.04333333333333332 radius=0.01
- link link12: mass 0.012499999999999999 -> 0.024999999999999998
- link link13: mass 0.012499999999999999 -> 0.024999999999999998; geometry collision cylinder length=0.04333333333333332 radius=0.01; visual cylinder length=0.04333333333333332 radius=0.01
- link link14: mass 0.012499999999999999 -> 0.024999999999999998
- link link15: mass 0.012499999999999999 -> 0.024999999999999998; geometry collision cylinder length=0.04333333333333332 radius=0.01; visual cylinder length=0.04333333333333332 radius=0.01
- link link16: mass 0.012499999999999999 -> 0.024999999999999998
- link link17: mass 0.012499999999999999 -> 0.024999999999999998; geometry collision cylinder length=0.04333333333333332 radius=0.01; visual cylinder length=0.04333333333333332 radius=0.01
- link link18: mass 0.012499999999999999 -> 0.024999999999999998
- link link19: mass 0.012499999999999999 -> 0.024999999999999998; geometry collision cylinder length=0.04333333333333332 radius=0.01; visual cylinder length=0.04333333333333332 radius=0.01
- link link2: mass 0.012499999999999999 -> 0.024999999999999998
- link link20: mass 0.012499999999999999 -> 0.024999999999999998
- link link21: mass 0.012499999999999999 -> 0.024999999999999998; geometry collision cylinder length=0.04333333333333332 radius=0.01; visual cylinder length=0.04333333333333332 radius=0.01
- link link22: mass 0.012499999999999999 -> 0.024999999999999998
- link link23: mass 0.012499999999999999 -> 0.024999999999999998; geometry collision cylinder length=0.04333333333333332 radius=0.01; visual cylinder length=0.04333333333333332 radius=0.01
- link link3: mass 0.012499999999999999 -> 0.024999999999999998; geometry collision cylinder length=0.04333333333333332 radius=0.01; visual cylinder length=0.04333333333333332 radius=0.01
- link link4: mass 0.012499999999999999 -> 0.024999999999999998
- link link5: mass 0.012499999999999999 -> 0.024999999999999998; geometry collision cylinder length=0.04333333333333332 radius=0.01; visual cylinder length=0.04333333333333332 radius=0.01
- link link6: mass 0.012499999999999999 -> 0.024999999999999998
- link link7: mass 0.012499999999999999 -> 0.024999999999999998; geometry collision cylinder length=0.04333333333333332 radius=0.01; visual cylinder length=0.04333333333333332 radius=0.01
- link link8: mass 0.012499999999999999 -> 0.024999999999999998
- link link9: mass 0.012499999999999999 -> 0.024999999999999998; geometry collision cylinder length=0.04333333333333332 radius=0.01; visual cylinder length=0.04333333333333332 radius=0.01
Joints:
- removed joint joint24
- removed joint joint25
- removed joint joint26
- removed joint joint27
- removed joint joint28
- removed joint joint29
- removed joint joint30
- removed joint joint31
- removed joint joint32
- removed joint joint33
- removed joint joint34
- removed joint joint35
- removed joint joint36
- removed joint joint37
- removed joint joint38
- removed joint joint39
- removed joint joint40
- removed joint joint41
- removed joint joint42
- removed joint joint43
- removed joint joint44
- removed joint joint45
- removed joint joint46
- removed joint joint47
- joint joint10: origin xyz=0.0 0.0 0.041666666666666664 -> xyz=0.0 0.0 0.06333333333333332
- joint joint12: origin xyz=0.0 0.0 0.041666666666666664 -> xyz=0.0 0.0 0.06333333333333332
- joint joint14: origin xyz=0.0 0.0 0.041666666666666664 -> xyz=0.0 0.0 0.06333333333333332
- joint joint16: origin xyz=0.0 0.0 0.041666666666666664 -> xyz=0.0 0.0 0.06333333333333332
- joint joint18: origin xyz=0.0 0.0 0.041666666666666664 -> xyz=0.0 0.0 0.06333333333333332
- joint joint2: origin xyz=0.0 0.0 0.041666666666666664 -> xyz=0.0 0.0 0.06333333333333332
- joint joint20: origin xyz=0.0 0.0 0.041666666666666664 -> xyz=0.0 0.0 0.06333333333333332
- joint joint22: origin xyz=0.0 0.0 0.041666666666666664 -> xyz=0.0 0.0 0.06333333333333332
- joint joint4: origin xyz=0.0 0.0 0.041666666666666664 -> xyz=0.0 0.0 0.06333333333333332
- joint joint6: origin xyz=0.0 0.0 0.041666666666666664 -> xyz=0.0 0.0 0.06333333333333332
- joint joint8: origin xyz=0.0 0.0 0.041666666666666664 -> xyz=0.0 0.0 0.06333333333333332

File: rope.urdf (robot description, URDF)
Before this commit: robot rope, 48 links, 48 joints
Links:
- removed link link24
- removed link link25
- removed link link26
- removed link link27
- removed link link28
- removed link link29
- removed link link30
- removed link link31
- removed link link32
- removed link link33
- removed link link34
- removed link link35
- removed link link36
- removed link link37
- removed link link38
- removed link link39
- removed link link40
- removed link link41
- removed link link42
- removed link link43
- removed link link44
- removed link link45
- removed link link46
- removed link link47
- link link0: mass 0.012499999999999999 -> 0.024999999999999998
- link link1: mass 0.012499999999999999 -> 0.024999999999999998; geometry collision cylinder length=0.04333333333333332 radius=0.01; visual cylinder length=0.04333333333333332 radius=0.01
- link link10: mass 0.012499999999999999 -> 0.024999999999999998
- link link11: mass 0.012499999999999999 -> 0.024999999999999998; geometry collision cylinder length=0.04333333333333332 radius=0.01; visual cylinder length=0.04333333333333332 radius=0.01
- link link12: mass 0.012499999999999999 -> 0.024999999999999998
- link link13: mass 0.012499999999999999 -> 0.024999999999999998; geometry collision cylinder length=0.04333333333333332 radius=0.01; visual cylinder length=0.04333333333333332 radius=0.01
- link link14: mass 0.012499999999999999 -> 0.024999999999999998
- link link15: mass 0.012499999999999999 -> 0.024999999999999998; geometry collision cylinder length=0.04333333333333332 radius=0.01; visual cylinder length=0.04333333333333332 radius=0.01
- link link16: mass 0.012499999999999999 -> 0.024999999999999998
- link link17: mass 0.012499999999999999 -> 0.024999999999999998; geometry collision cylinder length=0.04333333333333332 radius=0.01; visual cylinder length=0.04333333333333332 radius=0.01
- link link18: mass 0.012499999999999999 -> 0.024999999999999998
- link link19: mass 0.012499999999999999 -> 0.024999999999999998; geometry collision cylinder length=0.04333333333333332 radius=0.01; visual cylinder length=0.04333333333333332 radius=0.01
- link link2: mass 0.012499999999999999 -> 0.024999999999999998
- link link20: mass 0.012499999999999999 -> 0.024999999999999998
- link link21: mass 0.012499999999999999 -> 0.024999999999999998; geometry collision cylinder length=0.04333333333333332 radius=0.01; visual cylinder length=0.04333333333333332 radius=0.01
- link link22: mass 0.012499999999999999 -> 0.024999999999999998
- link link23: mass 0.012499999999999999 -> 0.024999999999999998; geometry collision cylinder length=0.04333333333333332 radius=0.01; visual cylinder length=0.04333333333333332 radius=0.01
- link link3: mass 0.012499999999999999 -> 0.024999999999999998; geometry collision cylinder length=0.04333333333333332 radius=0.01; visual cylinder length=0.04333333333333332 radius=0.01
- link link4: mass 0.012499999999999999 -> 0.024999999999999998
- link link5: mass 0.012499999999999999 -> 0.024999999999999998; geometry collision cylinder length=0.04333333333333332 radius=0.01; visual cylinder length=0.04333333333333332 radius=0.01
- link link6: mass 0.012499999999999999 -> 0.024999999999999998
- link link7: mass 0.012499999999999999 -> 0.024999999999999998; geometry collision cylinder length=0.04333333333333332 radius=0.01; visual cylinder length=0.04333333333333332 radius=0.01
- link link8: mass 0.012499999999999999 -> 0.024999999999999998
- link link9: mass 0.012499999999999999 -> 0.024999999999999998; geometry collision cylinder length=0.04333333333333332 radius=0.01; visual cylinder length=0.04333333333333332 radius=0.01
Joints:
- removed joint joint24
- removed joint joint25
- removed joint joint26
- removed joint joint27
- removed joint joint28
- removed joint joint29
- removed joint joint30
- removed joint joint31
- removed joint joint32
- removed joint joint33
- removed joint joint34
- removed joint joint35
- removed joint joint36
- removed joint joint37
- removed joint joint38
- removed joint joint39
- removed joint joint40
- removed joint joint41
- removed joint joint42
- removed joint joint43
- removed joint joint44
- removed joint joint45
- removed joint joint46
- removed joint joint47
- joint joint10: origin xyz=0.0 0.0 0.041666666666666664 -> xyz=0.0 0.0 0.06333333333333332
- joint joint12: origin xyz=0.0 0.0 0.041666666666666664 -> xyz=0.0 0.0 0.06333333333333332
- joint joint14: origin xyz=0.0 0.0 0.041666666666666664 -> xyz=0.0 0.0 0.06333333333333332
- joint joint16: origin xyz=0.0 0.0 0.041666666666666664 -> xyz=0.0 0.0 0.06333333333333332
- joint joint18: origin xyz=0.0 0.0 0.041666666666666664 -> xyz=0.0 0.0 0.06333333333333332
- joint joint2: origin xyz=0.0 0.0 0.041666666666666664 -> xyz=0.0 0.0 0.06333333333333332
- joint joint20: origin xyz=0.0 0.0 0.041666666666666664 -> xyz=0.0 0.0 0.06333333333333332
- joint joint22: origin xyz=0.0 0.0 0.041666666666666664 -> xyz=0.0 0.0 0.06333333333333332
- joint joint4: origin xyz=0.0 0.0 0.041666666666666664 -> xyz=0.0 0.0 0.06333333333333332
- joint joint6: origin xyz=0.0 0.0 0.041666666666666664 -> xyz=0.0 0.0 0.06333333333333332
- joint joint8: origin xyz=0.0 0.0 0.041666666666666664 -> xyz=0.0 0.0 0.06333333333333332
