Commit message: Working rope-end-static with summary writer. Failed to modify Rope prop.
Changing rope property leads to failure in dynamics.... We'll come back later.

File: assets/urdf/franka_description/robots/franka_panda_rope.urdf (robot description, URDF)
Before this commit: robot panda, 33 links, 32 joints
Links:
- added link link24, mass 0.012499999999999999; collision cylinder length=0 radius=0; visual cylinder length=0 radius=0
- added link link25, mass 0.012499999999999999; collision cylinder length=0.041666666666666664 radius=0.02; visual cylinder length=0.041666666666666664 radius=0.02
- added link link26, mass 0.012499999999999999; collision cylinder length=0 radius=0; visual cylinder length=0 radius=0
- added link link27, mass 0.012499999999999999; collision cylinder length=0.041666666666666664 radius=0.02; visual cylinder length=0.041666666666666664 radius=0.02
- added link link28, mass 0.012499999999999999; collision cylinder length=0 radius=0; visual cylinder length=0 radius=0
- added link link29, mass 0.012499999999999999; collision cylinder length=0.041666666666666664 radius=0.02; visual cylinder length=0.041666666666666664 radius=0.02
- added link link30, mass 0.012499999999999999; collision cylinder length=0 radius=0; visual cylinder length=0 radius=0
- added link link31, mass 0.012499999999999999; collision cylinder length=0.041666666666666664 radius=0.02; visual cylinder length=0.041666666666666664 radius=0.02
- added link link32, mass 0.012499999999999999; collision cylinder length=0 radius=0; visual cylinder length=0 radius=0
- added link link33, mass 0.012499999999999999; collision cylinder length=0.041666666666666664 radius=0.02; visual cylinder length=0.041666666666666664 radius=0.02
- added link link34, mass 0.012499999999999999; collision cylinder length=0 radius=0; visual cylinder length=0 radius=0
- added link link35, mass 0.012499999999999999; collision cylinder length=0.041666666666666664 radius=0.02; visual cylinder length=0.041666666666666664 radius=0.02
- added link link36, mass 0.012499999999999999; collision cylinder length=0 radius=0; visual cylinder length=0 radius=0
- added link link37, mass 0.012499999999999999; collision cylinder length=0.041666666666666664 radius=0.02; visual cylinder length=0.041666666666666664 radius=0.02
- added link link38, mass 0.012499999999999999; collision cylinder length=0 radius=0; visual cylinder length=0 radius=0
- added link link39, mass 0.012499999999999999; collision cylinder length=0.041666666666666664 radius=0.02; visual cylinder length=0.041666666666666664 radius=0.02
- added link link40, mass 0.012499999999999999; collision cylinder length=0 radius=0; visual cylinder length=0 radius=0
- added link link41, mass 0.012499999999999999; collision cylinder length=0.041666666666666664 radius=0.02; visual cylinder length=0.041666666666666664 radius=0.02
- added link link42, mass 0.012499999999999999; collision cylinder length=0 radius=0; visual cylinder length=0 radius=0
- added link link43, mass 0.012499999999999999; collision cylinder length=0.041666666666666664 radius=0.02; visual cylinder length=0.041666666666666664 radius=0.02
- added link link44, mass 0.012499999999999999; collision cylinder length=0 radius=0; visual cylinder length=0 radius=0
- added link link45, mass 0.012499999999999999; collision cylinder length=0.041666666666666664 radius=0.02; visual cylinder length=0.041666666666666664 radius=0.02
- added link link46, mass 0.012499999999999999; collision cylinder length=0 radius=0; visual cylinder length=0 radius=0
- added link link47, mass 0.012499999999999999; collision cylinder length=0.041666666666666664 radius=0.02; visual cylinder length=0.041666666666666664 radius=0.02
- link link0: mass 0.024999999999999998 -> 0.012499999999999999
- link link1: mass 0.024999999999999998 -> 0.012499999999999999; geometry collision cylinder length=0.041666666666666664 radius=0.02; visual cylinder length=0.041666666666666664 radius=0.02
- link link10: mass 0.024999999999999998 -> 0.012499999999999999
- link link11: mass 0.024999999999999998 -> 0.012499999999999999; geometry collision cylinder length=0.041666666666666664 radius=0.02; visual cylinder length=0.041666666666666664 radius=0.02
- link link12: mass 0.024999999999999998 -> 0.012499999999999999
- link link13: mass 0.024999999999999998 -> 0.012499999999999999; geometry collision cylinder length=0.041666666666666664 radius=0.02; visual cylinder length=0.041666666666666664 radius=0.02
- link link14: mass 0.024999999999999998 -> 0.012499999999999999
- link link15: mass 0.024999999999999998 -> 0.012499999999999999; geometry collision cylinder length=0.041666666666666664 radius=0.02; visual cylinder length=0.041666666666666664 radius=0.02
- link link16: mass 0.024999999999999998 -> 0.012499999999999999
- link link17: mass 0.024999999999999998 -> 0.012499999999999999; geometry collision cylinder length=0.041666666666666664 radius=0.02; visual cylinder length=0.041666666666666664 radius=0.02
- link link18: mass 0.024999999999999998 -> 0.012499999999999999
- link link19: mass 0.024999999999999998 -> 0.012499999999999999; geometry collision cylinder length=0.041666666666666664 radius=0.02; visual cylinder length=0.041666666666666664 radius=0.02
- link link2: mass 0.024999999999999998 -> 0.012499999999999999
- link link20: mass 0.024999999999999998 -> 0.012499999999999999
- link link21: mass 0.024999999999999998 -> 0.012499999999999999; geometry collision cylinder length=0.041666666666666664 radius=0.02; visual cylinder length=0.041666666666666664 radius=0.02
- link link22: mass 0.024999999999999998 -> 0.012499999999999999
- link link23: mass 0.024999999999999998 -> 0.012499999999999999; geometry collision cylinder length=0.041666666666666664 radius=0.02; visual cylinder length=0.041666666666666664 radius=0.02
- link link3: mass 0.024999999999999998 -> 0.012499999999999999; geometry collision cylinder length=0.041666666666666664 radius=0.02; visual cylinder length=0.041666666666666664 radius=0.02
- link link4: mass 0.024999999999999998 -> 0.012499999999999999
- link link5: mass 0.024999999999999998 -> 0.012499999999999999; geometry collision cylinder length=0.041666666666666664 radius=0.02; visual cylinder length=0.041666666666666664 radius=0.02
- link link6: mass 0.024999999999999998 -> 0.012499999999999999
- link link7: mass 0.024999999999999998 -> 0.012499999999999999; geometry collision cylinder length=0.041666666666666664 radius=0.02; visual cylinder length=0.041666666666666664 radius=0.02
- link link8: mass 0.024999999999999998 -> 0.012499999999999999
- link link9: mass 0.024999999999999998 -> 0.012499999999999999; geometry collision cylinder length=0.041666666666666664 radius=0.02; visual cylinder length=0.041666666666666664 radius=0.02
Joints:
- added joint joint24: type revolute, parent link23, child link24, origin xyz=0.0 0.0 0.041666666666666664, axis 0 1 0
- added joint joint25: type revolute, parent link24, child link25, origin xyz=0.0 0.0 0, axis 1 0 0
- added joint joint26: type revolute, parent link25, child link26, origin xyz=0.0 0.0 0.041666666666666664, axis 0 1 0
- added joint joint27: type revolute, parent link26, child link27, origin xyz=0.0 0.0 0, axis 1 0 0
- added joint joint28: type revolute, parent link27, child link28, origin xyz=0.0 0.0 0.041666666666666664, axis 0 1 0
- added joint joint29: type revolute, parent link28, child link29, origin xyz=0.0 0.0 0, axis 1 0 0
- added joint joint30: type revolute, parent link29, child link30, origin xyz=0.0 0.0 0.041666666666666664, axis 0 1 0
- added joint joint31: type revolute, parent link30, child link31, origin xyz=0.0 0.0 0, axis 1 0 0
- added joint joint32: type revolute, parent link31, child link32, origin xyz=0.0 0.0 0.041666666666666664, axis 0 1 0
- added joint joint33: type revolute, parent link32, child link33, origin xyz=0.0 0.0 0, axis 1 0 0
- added joint joint34: type revolute, parent link33, child link34, origin xyz=0.0 0.0 0.041666666666666664, axis 0 1 0
- added joint joint35: type revolute, parent link34, child link35, origin xyz=0.0 0.0 0, axis 1 0 0
- added joint joint36: type revolute, parent link35, child link36, origin xyz=0.0 0.0 0.041666666666666664, axis 0 1 0
- added joint joint37: type revolute, parent link36, child link37, origin xyz=0.0 0.0 0, axis 1 0 0
- added joint joint38: type revolute, parent link37, child link38, origin xyz=0.0 0.0 0.041666666666666664, axis 0 1 0
- added joint joint39: type revolute, parent link38, child link39, origin xyz=0.0 0.0 0, axis 1 0 0
- added joint joint40: type revolute, parent link39, child link40, origin xyz=0.0 0.0 0.041666666666666664, axis 0 1 0
- added joint joint41: type revolute, parent link40, child link41, origin xyz=0.0 0.0 0, axis 1 0 0
- added joint joint42: type revolute, parent link41, child link42, origin xyz=0.0 0.0 0.041666666666666664, axis 0 1 0
- added joint joint43: type revolute, parent link42, child link43, origin xyz=0.0 0.0 0, axis 1 0 0
- added joint joint44: type revolute, parent link43, child link44, origin xyz=0.0 0.0 0.041666666666666664, axis 0 1 0
- added joint joint45: type revolute, parent link44, child link45, origin xyz=0.0 0.0 0, axis 1 0 0
- added joint joint46: type revolute, parent link45, child link46, origin xyz=0.0 0.0 0.041666666666666664, axis 0 1 0
- added joint joint47: type revolute, parent link46, child link47, origin xyz=0.0 0.0 0, axis 1 0 0
- joint joint10: origin xyz=0.0 0.0 0.06333333333333332 -> xyz=0.0 0.0 0.041666666666666664
- joint joint12: origin xyz=0.0 0.0 0.06333333333333332 -> xyz=0.0 0.0 0.041666666666666664
- joint joint14: origin xyz=0.0 0.0 0.06333333333333332 -> xyz=0.0 0.0 0.041666666666666664
- joint joint16: origin xyz=0.0 0.0 0.06333333333333332 -> xyz=0.0 0.0 0.041666666666666664
- joint joint18: origin xyz=0.0 0.0 0.06333333333333332 -> xyz=0.0 0.0 0.041666666666666664
- joint joint2: origin xyz=0.0 0.0 0.06333333333333332 -> xyz=0.0 0.0 0.041666666666666664
- joint joint20: origin xyz=0.0 0.0 0.06333333333333332 -> xyz=0.0 0.0 0.041666666666666664
- joint joint22: origin xyz=0.0 0.0 0.06333333333333332 -> xyz=0.0 0.0 0.041666666666666664
- joint joint4: origin xyz=0.0 0.0 0.06333333333333332 -> xyz=0.0 0.0 0.041666666666666664
- joint joint6: origin xyz=0.0 0.0 0.06333333333333332 -> xyz=0.0 0.0 0.041666666666666664
- joint joint8: origin xyz=0.0 0.0 0.06333333333333332 -> xyz=0.0 0.0 0.041666666666666664

File: rope.urdf (robot description, URDF)
Before this commit: robot rope, 24 links, 24 joints
Links:
- added link link24, mass 0.012499999999999999; collision cylinder length=0 radius=0; visual cylinder length=0 radius=0
- added link link25, mass 0.012499999999999999; collision cylinder length=0.041666666666666664 radius=0.02; visual cylinder length=0.041666666666666664 radius=0.02
- added link link26, mass 0.012499999999999999; collision cylinder length=0 radius=0; visual cylinder length=0 radius=0
- added link link27, mass 0.012499999999999999; collision cylinder length=0.041666666666666664 radius=0.02; visual cylinder length=0.041666666666666664 radius=0.02
- added link link28, mass 0.012499999999999999; collision cylinder length=0 radius=0; visual cylinder length=0 radius=0
- added link link29, mass 0.012499999999999999; collision cylinder length=0.041666666666666664 radius=0.02; visual cylinder length=0.041666666666666664 radius=0.02
- added link link30, mass 0.012499999999999999; collision cylinder length=0 radius=0; visual cylinder length=0 radius=0
- added link link31, mass 0.012499999999999999; collision cylinder length=0.041666666666666664 radius=0.02; visual cylinder length=0.041666666666666664 radius=0.02
- added link link32, mass 0.012499999999999999; collision cylinder length=0 radius=0; visual cylinder length=0 radius=0
- added link link33, mass 0.012499999999999999; collision cylinder length=0.041666666666666664 radius=0.02; visual cylinder length=0.041666666666666664 radius=0.02
- added link link34, mass 0.012499999999999999; collision cylinder length=0 radius=0; visual cylinder length=0 radius=0
- added link link35, mass 0.012499999999999999; collision cylinder length=0.041666666666666664 radius=0.02; visual cylinder length=0.041666666666666664 radius=0.02
- added link link36, mass 0.012499999999999999; collision cylinder length=0 radius=0; visual cylinder length=0 radius=0
- added link link37, mass 0.012499999999999999; collision cylinder length=0.041666666666666664 radius=0.02; visual cylinder length=0.041666666666666664 radius=0.02
- added link link38, mass 0.012499999999999999; collision cylinder length=0 radius=0; visual cylinder length=0 radius=0
- added link link39, mass 0.012499999999999999; collision cylinder length=0.041666666666666664 radius=0.02; visual cylinder length=0.041666666666666664 radius=0.02
- added link link40, mass 0.012499999999999999; collision cylinder length=0 radius=0; visual cylinder length=0 radius=0
- added link link41, mass 0.012499999999999999; collision cylinder length=0.041666666666666664 radius=0.02; visual cylinder length=0.041666666666666664 radius=0.02
- added link link42, mass 0.012499999999999999; collision cylinder length=0 radius=0; visual cylinder length=0 radius=0
- added link link43, mass 0.012499999999999999; collision cylinder length=0.041666666666666664 radius=0.02; visual cylinder length=0.041666666666666664 radius=0.02
- added link link44, mass 0.012499999999999999; collision cylinder length=0 radius=0; visual cylinder length=0 radius=0
- added link link45, mass 0.012499999999999999; collision cylinder length=0.041666666666666664 radius=0.02; visual cylinder length=0.041666666666666664 radius=0.02
- added link link46, mass 0.012499999999999999; collision cylinder length=0 radius=0; visual cylinder length=0 radius=0
- added link link47, mass 0.012499999999999999; collision cylinder length=0.041666666666666664 radius=0.02; visual cylinder length=0.041666666666666664 radius=0.02
- link link0: mass 0.024999999999999998 -> 0.012499999999999999
- link link1: mass 0.024999999999999998 -> 0.012499999999999999; geometry collision cylinder length=0.041666666666666664 radius=0.02; visual cylinder length=0.041666666666666664 radius=0.02
- link link10: mass 0.024999999999999998 -> 0.012499999999999999
- link link11: mass 0.024999999999999998 -> 0.012499999999999999; geometry collision cylinder length=0.041666666666666664 radius=0.02; visual cylinder length=0.041666666666666664 radius=0.02
- link link12: mass 0.024999999999999998 -> 0.012499999999999999
- link link13: mass 0.024999999999999998 -> 0.012499999999999999; geometry collision cylinder length=0.041666666666666664 radius=0.02; visual cylinder length=0.041666666666666664 radius=0.02
- link link14: mass 0.024999999999999998 -> 0.012499999999999999
- link link15: mass 0.024999999999999998 -> 0.012499999999999999; geometry collision cylinder length=0.041666666666666664 radius=0.02; visual cylinder length=0.041666666666666664 radius=0.02
- link link16: mass 0.024999999999999998 -> 0.012499999999999999
- link link17: mass 0.024999999999999998 -> 0.012499999999999999; geometry collision cylinder length=0.041666666666666664 radius=0.02; visual cylinder length=0.041666666666666664 radius=0.02
- link link18: mass 0.024999999999999998 -> 0.012499999999999999
- link link19: mass 0.024999999999999998 -> 0.012499999999999999; geometry collision cylinder length=0.041666666666666664 radius=0.02; visual cylinder length=0.041666666666666664 radius=0.02
- link link2: mass 0.024999999999999998 -> 0.012499999999999999
- link link20: mass 0.024999999999999998 -> 0.012499999999999999
- link link21: mass 0.024999999999999998 -> 0.012499999999999999; geometry collision cylinder length=0.041666666666666664 radius=0.02; visual cylinder length=0.041666666666666664 radius=0.02
- link link22: mass 0.024999999999999998 -> 0.012499999999999999
- link link23: mass 0.024999999999999998 -> 0.012499999999999999; geometry collision cylinder length=0.041666666666666664 radius=0.02; visual cylinder length=0.041666666666666664 radius=0.02
- link link3: mass 0.024999999999999998 -> 0.012499999999999999; geometry collision cylinder length=0.041666666666666664 radius=0.02; visual cylinder length=0.041666666666666664 radius=0.02
- link link4: mass 0.024999999999999998 -> 0.012499999999999999
- link link5: mass 0.024999999999999998 -> 0.012499999999999999; geometry collision cylinder length=0.041666666666666664 radius=0.02; visual cylinder length=0.041666666666666664 radius=0.02
- link link6: mass 0.024999999999999998 -> 0.012499999999999999
- link link7: mass 0.024999999999999998 -> 0.012499999999999999; geometry collision cylinder length=0.041666666666666664 radius=0.02; visual cylinder length=0.041666666666666664 radius=0.02
- link link8: mass 0.024999999999999998 -> 0.012499999999999999
- link link9: mass 0.024999999999999998 -> 0.012499999999999999; geometry collision cylinder length=0.041666666666666664 radius=0.02; visual cylinder length=0.041666666666666664 radius=0.02
Joints:
- added joint joint24: type revolute, parent link23, child link24, origin xyz=0.0 0.0 0.041666666666666664, axis 0 1 0
- added joint joint25: type revolute, parent link24, child link25, origin xyz=0.0 0.0 0, axis 1 0 0
- added joint joint26: type revolute, parent link25, child link26, origin xyz=0.0 0.0 0.041666666666666664, axis 0 1 0
- added joint joint27: type revolute, parent link26, child link27, origin xyz=0.0 0.0 0, axis 1 0 0
- added joint joint28: type revolute, parent link27, child link28, origin xyz=0.0 0.0 0.041666666666666664, axis 0 1 0
- added joint joint29: type revolute, parent link28, child link29, origin xyz=0.0 0.0 0, axis 1 0 0
- added joint joint30: type revolute, parent link29, child link30, origin xyz=0.0 0.0 0.041666666666666664, axis 0 1 0
- added joint joint31: type revolute, parent link30, child link31, origin xyz=0.0 0.0 0, axis 1 0 0
- added joint joint32: type revolute, parent link31, child link32, origin xyz=0.0 0.0 0.041666666666666664, axis 0 1 0
- added joint joint33: type revolute, parent link32, child link33, origin xyz=0.0 0.0 0, axis 1 0 0
- added joint joint34: type revolute, parent link33, child link34, origin xyz=0.0 0.0 0.041666666666666664, axis 0 1 0
- added joint joint35: type revolute, parent link34, child link35, origin xyz=0.0 0.0 0, axis 1 0 0
- added joint joint36: type revolute, parent link35, child link36, origin xyz=0.0 0.0 0.041666666666666664, axis 0 1 0
- added joint joint37: type revolute, parent link36, child link37, origin xyz=0.0 0.0 0, axis 1 0 0
- added joint joint38: type revolute, parent link37, child link38, origin xyz=0.0 0.0 0.041666666666666664, axis 0 1 0
- added joint joint39: type revolute, parent link38, child link39, origin xyz=0.0 0.0 0, axis 1 0 0
- added joint joint40: type revolute, parent link39, child link40, origin xyz=0.0 0.0 0.041666666666666664, axis 0 1 0
- added joint joint41: type revolute, parent link40, child link41, origin xyz=0.0 0.0 0, axis 1 0 0
- added joint joint42: type revolute, parent link41, child link42, origin xyz=0.0 0.0 0.041666666666666664, axis 0 1 0
- added joint joint43: type revolute, parent link42, child link43, origin xyz=0.0 0.0 0, axis 1 0 0
- added joint joint44: type revolute, parent link43, child link44, origin xyz=0.0 0.0 0.041666666666666664, axis 0 1 0
- added joint joint45: type revolute, parent link44, child link45, origin xyz=0.0 0.0 0, axis 1 0 0
- added joint joint46: type revolute, parent link45, child link46, origin xyz=0.0 0.0 0.041666666666666664, axis 0 1 0
- added joint joint47: type revolute, parent link46, child link47, origin xyz=0.0 0.0 0, axis 1 0 0
- joint joint10: origin xyz=0.0 0.0 0.06333333333333332 -> xyz=0.0 0.0 0.041666666666666664
- joint joint12: origin xyz=0.0 0.0 0.06333333333333332 -> xyz=0.0 0.0 0.041666666666666664
- joint joint14: origin xyz=0.0 0.0 0.06333333333333332 -> xyz=0.0 0.0 0.041666666666666664
- joint joint16: origin xyz=0.0 0.0 0.06333333333333332 -> xyz=0.0 0.0 0.041666666666666664
- joint joint18: origin xyz=0.0 0.0 0.06333333333333332 -> xyz=0.0 0.0 0.041666666666666664
- joint joint2: origin xyz=0.0 0.0 0.06333333333333332 -> xyz=0.0 0.0 0.041666666666666664
- joint joint20: origin xyz=0.0 0.0 0.06333333333333332 -> xyz=0.0 0.0 0.041666666666666664
- joint joint22: origin xyz=0.0 0.0 0.06333333333333332 -> xyz=0.0 0.0 0.041666666666666664
- joint joint4: origin xyz=0.0 0.0 0.06333333333333332 -> xyz=0.0 0.0 0.041666666666666664
- joint joint6: origin xyz=0.0 0.0 0.06333333333333332 -> xyz=0.0 0.0 0.041666666666666664
- joint joint8: origin xyz=0.0 0.0 0.06333333333333332 -> xyz=0.0 0.0 0.041666666666666664
